File: Wheel-Control-Board-Design/BoardV1Proto/BoardV1Proto.kicad_sch (KiCad schematic)
At the start: 15 parts

Commit message: First commit to back up
Parts:
- removed U?: ESP32-WROOM-32, RF_Module:ESP32-WROOM-32, symbol RF_Module:ESP32-WROOM-32
- added D?: LED, symbol Device:LED
- added R?: R, symbol Device:R
- added SW?: SW_Push, symbol Switch:SW_Push
Connections:
- net +3V3: now also U?.1 (3V3), U?.2 (CHIP_PU), R?.2, SW?.2
- net GND: now also U?.38 (GND), R?.1
- net LCD Mode Button: now reaches SW?.1
- net LCD Mode Button: now also U?.5 (VDET_1/GPIO34/ADC1_CH6)
- net Coast Regen: now reaches U?.3 (SENSOR_VP/GPIO36/ADC1_CH0)
- net Coast Regen: now also RV?.2
- net Brake Regen: now reaches U?.4 (SENSOR_VN/GPIO39/ADC1_CH3)
- net Brake Regen: now also RV?.2
- net Drive Mode Select: now reaches U?.6 (VDET_2/GPIO35/ADC1_CH7)
- net Drive Mode Select: now also SW?.1
- net RTD Button: now reaches U?.7 (32K_XP/GPIO32/ADC1_CH4)
- net RTD Button: now also SW?.1
- net RTD Button LED: now reaches U?.8 (32K_XN/GPIO33/ADC1_CH5)
Other:
- moved on the sheet: R?, RV?, SW?
