File: Front-Control-Board/Front-Control-Board-Design/Front Board/Front Board.kicad_pcb (KiCad board)
At the start: 2 copper layers, 85.2 x 70.7 mm, 27 parts, among them J1 Conn_01x14, J2 Conn_01x14, J3 Conn_01x08, Q1 2N7002, U1 MAX33054EASA+T, U2 TS2940CP33 ROG, U3 ESP32-DevKitC

Commit message: oops forgot to push for awile
Routing:
- net VDD: track 154.8 -> 188.8 mm
- removed copper zone on B.Cu, net VDD
Other:
- board text added: "Front Board V2 C.Grund 17.2023"
Changed lines of the file:
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@@
       (drillshape 0)
       (scaleselection 1)
-      (outputdirectory "../../../BOARD GERBER/V1/Front/")
+      (outputdirectory "../../../BOARD GERBER/V2/Front/")
     )
   )
@@
   (gr_line (start 188.292956 111.524481) (end 172.807044 111.535519) (layer "Edge.Cuts") (width 0.1))
   (gr_arc (start 168.55184 115.785519) (mid 169.8 112.78) (end 172.807044 111.535519) (layer "Edge.Cuts") (width 0.1))
+  (gr_text "Front Board V2\nC.Grund 17.2023\n" (at 122.25 111.5) (layer "F.SilkS")
+    (effects (font (size 1.5 1.5) (thickness 0.3)))
+  )
   (segment (start 118.5 109.863817) (end 109.187989 100.551806) (width 0.8) (layer "B.Cu") (net 1))
   (segment (start 109.187989 100.551806) (end 109.187989 82.442011) (width 0.8) (layer "B.Cu") (net 1))
@@
   (segment (start 137.6 69.43) (end 137.6 70.67) (width 0.3) (layer "B.Cu") (net 3))
   (segment (start 125.1 75.93) (end 130.425 70.605) (width 0.8) (layer "B.Cu") (net 3))
+  (segment (start 130.425 70.605) (end 133.8125 67.2175) (width 0.3) (layer "B.Cu") (net 3))
   (segment (start 116.674521 102.170704) (end 116.674521 106.624804) (width 0.8) (layer "B.Cu") (net 3))
   (segment (start 115.1 82.53) (end 115.1 80.673845) (width 0.8) (layer "B.Cu") (net 3))
@@
   (segment (start 168.4 74.43) (end 169.765 75.795) (width 0.3) (layer "B.Cu") (net 3))
   (segment (start 170.924898 77.595) (end 172.194898 76.325) (width 0.3) (layer "B.Cu") (net 3))
+  (segment (start 137.535 70.605) (end 137.6 70.67) (width 0.3) (layer "B.Cu") (net 3))
+  (segment (start 130.36 70.67) (end 137.6 70.67) (width 1) (layer "B.Cu") (net 3))
   (segment (start 172.194898 76.325) (end 172.675 76.325) (width 0.3) (layer "B.Cu") (net 3))
   (segment (start 168.6 74.43) (end 169.69 73.34) (width 0.3) (layer "B.Cu") (net 3))
   (segment (start 169.69 73.34) (end 165.78 69.43) (width 0.3) (layer "B.Cu") (net 3))
   (segment (start 169.765 75.795) (end 169.765 77.595) (width 0.3) (layer "B.Cu") (net 3))
+  (segment (start 126.89 74.14) (end 132.9 68.13) (width 0.8) (layer "B.Cu") (net 3))
   (segment (start 137.6 69.43) (end 137.6 68.13) (width 0.3) (layer "B.Cu") (net 3))
   (segment (start 120.5 127.63) (end 118.5 129.63) (width 0.8) (layer "B.Cu") (net 3))
@@
   (segment (start 113.187989 98.684172) (end 116.674521 102.170704) (width 0.8) (layer "B.Cu") (net 3))
   (segment (start 170.69 74.34) (end 169.69 73.34) (width 0.3) (layer "B.Cu") (net 3))
+  (segment (start 132.9 68.13) (end 137.6 68.13) (width 1) (layer "B.Cu") (net 3))
+  (segment (start 133.8125 67.2175) (end 133.8125 65.93) (width 0.3) (layer "B.Cu") (net 3))
   (segment (start 170.69 74.34) (end 172.79 74.34) (width 0.3) (layer "B.Cu") (net 3))
   (segment (start 126.5 116.450283) (end 116.674521 106.624804) (width 0.8) (layer "B.Cu") (net 3))
   (segment (start 165.78 69.43) (end 137.6 69.43) (width 0.3) (layer "B.Cu") (net 3))
+  (segment (start 126.89 74.14) (end 130.36 70.67) (width 0.8) (layer "B.Cu") (net 3))
   (segment (start 113.187989 84.442011) (end 113.187989 98.684172) (width 0.8) (layer "B.Cu") (net 3))
+  (segment (start 125.1 75.93) (end 126.89 74.14) (width 0.8) (layer "B.Cu") (net 3))
   (segment (start 133 75.33) (end 133 73.18) (width 0.3) (layer "B.Cu") (net 3))
   (segment (start 179.20048 78.41798) (end 178.3625 77.58) (width 0.2) (layer "B.Cu") (net 4))
@@
       )
     )
-  )
-  (zone (net 3) (net_name "VDD") (layer "B.Cu") (hatch edge 0.508)
-    (connect_pads yes (clearance 0.508))
-    (min_thickness 0.254) (filled_areas_thickness no)
-    (fill yes (thermal_gap 0.508) (thermal_bridge_width 0.508))
-    (polygon
-      (pts
-        (xy 138.8 71.63)
-        (xy 135.8 71.63)
-        (xy 133.8 73.93)
-        (xy 127 73.83)
-        (xy 127 67.53)
-        (xy 138.8 67.13)
-      )
-    )

Commit message: V3
Parts:
- U2: value TS2940CP33 ROG -> TS2940CP33_ROG; moved to F.Cu
- moved C1 8.59 mm to (117.2, 68.6)
- moved D7 8.59 mm to (117.3, 66.8)
- moved C2 3.94 mm to (130.8, 71.6), turned to 90 degrees
- moved U2 2.62 mm to (126.2, 69.0), turned to 90 degrees
- moved R2 0.88 mm to (133.0, 65.0)
- moved D2 0.88 mm to (133.0, 63.2)
Connections:
- U2 pad 1: GND -> +12V
- U2 pad 2: VDD -> GND
- U2 pad 3: +12V -> VDD
Routing:
- net VDD: track 188.8 -> 177.3 mm
- net +12V: track 72.3 -> 83.1 mm
- net GND: vias 10 -> 11
