File: Front-Control-Board/Front-Control-Board-Design/Front Board/Front Board.kicad_sch (KiCad schematic)
At the start: 27 parts, among them J1 Conn_01x14, J2 Conn_01x14, J3 Conn_01x08, Q1 2N7002, U1 MAX33054EASA+T, U2 TS2940CP33 ROG, U3 ESP32-DevKitC

Commit message: V3
Parts:
- removed U2: TS2940CP33 ROG, Package_TO_SOT_SMD:TO-252-2, symbol Regulator_Linear:NCP1117-5.0_TO252
- added U2: TS2940CP33_ROG, Package_TO_SOT_SMD:TO-252-2, symbol AERO_Symbols:TS2940CP33_ROG
Connections:
- net +12V: now also U2.1 (VI)
- net GND: now also U2.2 (GND)
- net VDD: now also U2.3 (Vo)
Changed lines of the file:
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@@
     (stroke (width 0) (type default) (color 0 0 0 0))
   )
-  (wire (pts (xy 49.784 41.148) (xy 49.784 46.228))
+  (wire (pts (xy 49.53 40.64) (xy 49.53 45.72))
     (stroke (width 0) (type default) (color 0 0 0 0))
   )
@@
     (stroke (width 0) (type default) (color 0 0 0 0))
   )
+  (wire (pts (xy 49.53 45.72) (xy 49.784 46.228))
+    (stroke (width 0) (type default) (color 0 0 0 0))
+  )
   (wire (pts (xy 157.48 100.965) (xy 175.514 100.965))
     (stroke (width 0) (type default) (color 0 0 0 0))
@@
     (stroke (width 0) (type default) (color 0 0 0 0))
   )
-  (wire (pts (xy 33.274 33.528) (xy 42.164 33.528))
+  (wire (pts (xy 33.655 33.02) (xy 42.545 33.02))
     (stroke (width 0) (type default) (color 0 0 0 0))
   )
@@
     (stroke (width 0) (type default) (color 0 0 0 0))
   )
+  (wire (pts (xy 49.53 40.64) (xy 50.165 40.64))
+    (stroke (width 0) (type default) (color 0 0 0 0))
+  )
   (wire (pts (xy 181.356 77.343) (xy 181.356 79.883))
     (stroke (width 0) (type default) (color 0 0 0 0))
@@
     (stroke (width 0) (type default) (color 0 0 0 0))
   )
+  (wire (pts (xy 33.655 33.02) (xy 33.274 33.528))
+    (stroke (width 0) (type default) (color 0 0 0 0))
+  )
   (wire (pts (xy 81.534 173.99) (xy 80.01 173.99))
     (stroke (width 0) (type default) (color 0 0 0 0))
@@
     (stroke (width 0) (type default) (color 0 0 0 0))
   )
-  (wire (pts (xy 57.404 33.528) (xy 65.024 33.528))
+  (wire (pts (xy 57.785 33.02) (xy 65.405 33.02))
     (stroke (width 0) (type default) (color 0 0 0 0))
   )
@@
   )
   (wire (pts (xy 79.502 41.148) (xy 79.502 46.228))
+    (stroke (width 0) (type default) (color 0 0 0 0))
+  )
+  (wire (pts (xy 65.405 33.02) (xy 65.024 33.528))
     (stroke (width 0) (type default) (color 0 0 0 0))
   )
@@
     (pin "2")
   )
+  (symbol (lib_id "AERO_Symbols:TS2940CP33_ROG") (at 50.165 33.02 0) (unit 1)
+    (in_bom yes) (on_board yes) (fields_autoplaced)
+    (property "Reference" "U2" (id 0) (at 50.165 25.4 0))
+    (property "Value" "TS2940CP33_ROG" (id 1) (at 50.165 27.94 0))
+    (property "Footprint" "Package_TO_SOT_SMD:TO-252-2" (id 2) (at 50.165 33.02 0)
+      (effects (font (size 1.27 1.27)) hide)
+    )
+    (property "Datasheet" "" (id 3) (at 50.165 33.02 0)
+      (effects (font (size 1.27 1.27)) hide)
+    )
+    (pin "1")
+    (pin "2")
+    (pin "3")
+  )
   (symbol (lib_id "power:VDD") (at 81.915 75.565 0) (unit 1)
     (in_bom yes) (on_board yes) (fields_autoplaced)
@@
     (pin "1")
   )
-  (symbol (lib_id "Regulator_Linear:NCP1117-5.0_TO252") (at 49.784 33.528 0) (unit 1)
-    (in_bom yes) (on_board yes) (fields_autoplaced)
-    (property "Reference" "U2" (id 0) (at 49.784 27.6565 0))
-    (property "Value" "TS2940CP33 ROG" (id 1) (at 49.784 30.4316 0))
-    (property "Footprint" "Package_TO_SOT_SMD:TO-252-2" (id 2) (at 49.784 27.813 0)
-      (effects (font (size 1.27 1.27)) hide)
-    )
-    (property "Datasheet" "https://www.taiwansemi.com/assets/uploads/datasheet/TS2940_D15.pdf" (id 3) (at 49.784 33.528 0)
-      (effects (font (size 1.27 1.27)) hide)
-    )
-    (pin "1")
-    (pin "2")
-    (pin "3")
-  )
   (symbol (lib_id "power:GND") (at 73.025 158.115 0) (unit 1)
     (in_bom yes) (on_board yes)
@@
       (reference "U1") (unit 1) (value "MAX33054EASA+T") (footprint "AERO_Footprints:SOIC127P600X175-8N")
     )
-    (path "/de613e64-a694-40f1-9848-99e26219228a"
-      (reference "U2") (unit 1) (value "TS2940CP33 ROG") (footprint "Package_TO_SOT_SMD:TO-252-2")
+    (path "/7b22b3c7-87af-4c06-91e6-d5b323c7430d"
+      (reference "U2") (unit 1) (value "TS2940CP33_ROG") (footprint "Package_TO_SOT_SMD:TO-252-2")
     )
     (path "/12a6a643-8d09-4828-9fdd-0e9da0628c48"

Commit message: end of year DUMP
Other:
- note added: "Amp - seal connectors"
- note added: "Micro-Controler"
- note added: "Power Converter"
- moved on the sheet: C1, C2, D2, D3, D4, D5, D6, D7, J1, J2, J3, Q1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
