File: Rear-Control-Board/rear-control-board-Design/FuseBank.kicad_sch (KiCad schematic)
At the start: 10 parts

Commit message: V3
Connections:
- net +12V: no longer F9.1
- new net BATT_12: F9.1
Changed lines of the file:
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@@
   (junction (at 74.93 66.675) (diameter 0) (color 0 0 0 0)
   )
-  (junction (at 74.93 104.14) (diameter 0) (color 0 0 0 0)
-  )
   (junction (at 74.93 85.725) (diameter 0) (color 0 0 0 0)
   )
@@
   )
   (wire (pts (xy 74.93 98.425) (xy 74.93 104.14))
-    (stroke (width 0) (type default) (color 0 0 0 0))
-  )
-  (wire (pts (xy 74.93 104.14) (xy 74.93 110.49))
     (stroke (width 0) (type default) (color 0 0 0 0))
   )
@@
     )
   )
+  (global_label "BATT_12" (shape input) (at 74.93 110.49 180) (fields_autoplaced)
+    (effects (font (size 1.27 1.27)) (justify right))
+    (property "Intersheet References" "${INTERSHEET_REFS}" (id 0) (at 64.9253 110.4106 0)
+      (effects (font (size 1.27 1.27)) (justify right) hide)
+    )
+  )
