File: Rear-Control-Board/rear-control-board-Design/rear-control-board.kicad_pcb (KiCad board)
At the start: 2 copper layers, 139.1 x 102.8 mm, 55 parts, among them J1 Conn_01x23, J2 Conn_01x23, J3 Conn_01x08, J4 JST-B2B-VERT-2PIN, J5 JST-B2B-VERT-2PIN, J6 Conn_01x02, J7 Micro_SD_Card, K1 T9VV1K15-12S, K2 G5V-2, K3 G5V-2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

Commit message: oops forgot to push for awile
Routing:
- net /BATT_12V: track 11.9 -> 184.1 mm
- net /RINE_12: track 3.35 -> 162.1 mm
- net +12V: track 95.6 -> 168.3 mm
- net /PUMP_12V: track 3.20 -> 49.6 mm
- net /FAN_12V: track 0.00 -> 40.4 mm
- net /DCDC_IN: track 50.5 -> 88.1 mm
- net /FAN_RTRN_12V: track 12.4 -> 30.4 mm
- net /PUMP_RTRN_12V: track 34.5 -> 44.9 mm
- removed copper zone on B.Cu, net +12V
- removed copper zone on B.Cu, net /BATT_12V
- removed copper zone on B.Cu, net /DCDC_IN
- removed copper zone on B.Cu, net /FAN_12V
- removed copper zone on F.Cu, net /FAN_RTRN_12V
- removed copper zone on B.Cu, net /PUMP_12V
- removed copper zone on F.Cu, net /PUMP_RTRN_12V
- removed copper zone on B.Cu, net /RINE_12
Other:
- board text added: "RCB V2 C.Grund 17.2023"

Commit message: V3
Parts:
- removed Q2, Q3, Q4: PSMN5R2-60YL, Package_TO_SOT_SMD:LFPAK56
- added JP1: SolderJumper_2_Open, Jumper:SolderJumper-2_P1.3mm_Open_TrianglePad1.0x1.5mm, B.Cu at (148.5, 82.5)
- added K4: G5V-1, Relay_THT:Relay_SPDT_Omron_G5V-1, F.Cu at (75.3, 68.1)
- added K5: G5V-1, Relay_THT:Relay_SPDT_Omron_G5V-1, F.Cu at (75.5, 91.7)
- added K6: G5V-1, Relay_THT:Relay_SPDT_Omron_G5V-1, F.Cu at (85.0, 75.2)
- added Q1: 2N7002, Package_TO_SOT_SMD:SOT-23, F.Cu at (148.5, 86.2)
- added R1: 100k, Resistor_SMD:R_0603_1608Metric_Pad0.98x0.95mm_HandSolder, F.Cu at (140.5, 86.2)
- added R9: 2.2K, Resistor_SMD:R_0603_1608Metric_Pad0.98x0.95mm_HandSolder, F.Cu at (142.2, 88.2)
- C13, C2, C3: moved to B.Cu
- R3: value 10k -> 10K
- U2: value TS2940CP33 ROG -> TS2940CP33_ROG
- moved H1 158.4 mm to (182.5, 85.0)
- moved H2 111.3 mm to (70.5, 155.8)
- moved F9 20.0 mm to (86.0, 119.0)
- moved R8 15.4 mm to (147.0, 117.2)
- moved F10 14.1 mm to (126.0, 119.3), turned to 0 degrees
- moved C3 13.8 mm to (87.0, 95.5), turned to 180 degrees
- moved K1 10.2 mm to (96.7, 144.3)
- moved F3 8.75 mm to (105.8, 119.3)
- moved R5 7.63 mm to (144.0, 117.2)
- moved D11 7.26 mm to (90.7, 80.3), turned to 90 degrees
- moved D10 7.01 mm to (90.8, 91.5), turned to 90 degrees
- moved D12 6.74 mm to (90.8, 68.0), turned to 90 degrees
- moved R3 6.59 mm to (138.8, 88.2), turned to 90 degrees
- moved C13 3.20 mm to (77.8, 76.0)
- moved C2 3.20 mm to (73.0, 65.5)
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Connections:
- D3 pad 1: /BATT_12V -> BATT_12
- D3 pad 3: /BATT_12V -> BATT_12
- D4 pad 1: INT_12V -> Net-(D4-Pad1)
- D4 pad 2: /FAULT_LATCHER/BMS_SWITCH -> GND
- D7 pad 1: /FAULT_LATCHER/BMS_SWITCH -> /Controller/FAULT_BMS
- F9 pad 1: +12V -> BATT_12
- J1 pad 12: /BATT_12V -> BATT_12
- J1 pad 13: /BATT_12V -> BATT_12
- J1 pad 14: /BATT_12V -> BATT_12
- J1 pad 15: /BATT_12V -> BATT_12
- J4 pad 1: /FAULT_LATCHER/BMS_SWITCH -> INT_12V
- J4 pad 2: GND -> Net-(D4-Pad1)
- K1 pad 3: /BATT_12V -> BATT_12
- K2 pad 1: /FAULT_LATCHER/BMS_SWITCH -> Net-(D4-Pad1)
- K2 pad 13: Net-(K2-Pad13) -> /BRB_RTN
- K2 pad 16: INT_12V -> GND
- K2 pad 8: /FAULT_LATCHER/BMS_SWITCH -> Net-(D4-Pad1)
- K2 pad 9: /BRB_RTN -> Net-(K2-Pad9)
- K3 pad 9: Net-(K2-Pad13) -> Net-(K2-Pad9)
- R3 pad 1: VDD -> Net-(D4-Pad1)
- R3 pad 2: /FAULT_LATCHER/BMS_SWITCH -> Net-(JP1-Pad2)
- U1 pad 8: /FAULT_LATCHER/BMS_SWITCH -> /Controller/FAULT_BMS
- U2 pad 1: GND -> INT_12V
- U2 pad 2: VDD -> GND
- U2 pad 3: INT_12V -> VDD
Routing:
- net BATT_12: track 0.00 -> 572.8 mm, vias 0 -> 9
- net +12V: track 168.3 -> 495.5 mm
- net /BATT_12V: track 184.1 -> 0.00 mm
- net /FAULT_LATCHER/BMS_SWITCH: track 90.7 -> 0.00 mm, vias 1 -> 0
- net /PUMP_RTRN_12V: track 44.9 -> 121.4 mm, vias 0 -> 1
- net /Controller/FAULT_BMS: track 0.00 -> 73.7 mm, vias 0 -> 2
- net Net-(D4-Pad1): track 0.00 -> 39.5 mm
- net /PUMP_12V: track 49.6 -> 89.0 mm
- net /FAN_RTRN_12V: track 30.4 -> 62.0 mm
- net /RINE_12: track 162.1 -> 140.9 mm
- net /BRB_LOOP: track 47.6 -> 67.9 mm, vias 0 -> 1
- net Net-(K2-Pad9): track 0.00 -> 19.6 mm
- net Net-(JP1-Pad2): track 0.00 -> 17.7 mm, vias 0 -> 1
- net /Controller/FAN_CTRL: track 127.1 -> 141.7 mm
- net /FAN_12V: track 40.4 -> 54.5 mm
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Other:
- board size 139.1 x 102.8 mm -> 139 x 104.8 mm
- board text added: "RCB V2 C.Grund 52.2023"
- board text removed: "RCB V2 C.Grund 17.2023"

Commit message: OOPSIE
Parts:
- moved U1 21.8 mm to (183.2, 117.7)
- moved D5 21.8 mm to (135.0, 87.6)
- moved J5 21.8 mm to (142.4, 86.4)
- moved K2 21.8 mm to (129.8, 72.6)
- moved K3 21.8 mm to (111.8, 92.7)
- moved J6 21.8 mm to (145.8, 124.1)
- moved F10 21.8 mm to (119.3, 98.6)
- moved F3 21.8 mm to (99.1, 98.6)
- moved F9 21.8 mm to (79.3, 98.3)
- moved C12 21.8 mm to (143.7, 102.5)
- moved C3 21.8 mm to (80.3, 74.8)
- moved C4 21.8 mm to (105.9, 64.5)
- moved C8 21.8 mm to (138.5, 103.6)
- moved D10 21.8 mm to (84.0, 70.8)
- moved D11 21.8 mm to (84.0, 59.6)
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Connections:
- net /Controller/CLK renamed /Controller/SD_CLK
- J2 pad 11: unconnected-(J2-Pad11) -> PAC1_1
- J2 pad 12: unconnected-(J2-Pad12) -> PAC1_2
- J2 pad 13: unconnected-(J2-Pad13) -> PAC2_1
- J2 pad 14: unconnected-(J2-Pad14) -> PAC2_2
- J2 pad 3: unconnected-(J2-Pad3) -> BMS_Therm_Out
- J7 pad 1: /Controller/DAT2 -> unconnected-(J7-Pad1)
- J7 pad 2: /Controller/DAT3 -> /Controller/CS_SD
- J7 pad 3: /Controller/CMD -> /Controller/SD_MOSI
- J7 pad 7: /Controller/DAT0 -> /Controller/SD_MISO
- J7 pad 8: /Controller/DAT1 -> unconnected-(J7-Pad8)
- U1 pad 10: /Controller/FAN_CTRL -> PAC1_2
- U1 pad 11: unconnected-(U1-Pad11) -> PAC1_1
- U1 pad 13: /Controller/DAT2 -> /Controller/SD_MISO
- U1 pad 15: /Controller/DAT3 -> /Controller/SD_MOSI
- U1 pad 23: /Controller/CMD -> /Controller/CS_SD
- U1 pad 24: /Controller/DAT0 -> unconnected-(U1-Pad24)
- U1 pad 26: /Controller/DAT1 -> PAC2_2
- U1 pad 27: unconnected-(U1-Pad27) -> /Controller/BRAKE_CTRL
- U1 pad 33: unconnected-(U1-Pad33) -> /Controller/FAN_CTRL
- U1 pad 36: unconnected-(U1-Pad36) -> BMS_Therm_Out
- U1 pad 9: /Controller/BRAKE_CTRL -> PAC2_1
Routing:
- net /Controller/DAT0: track 87.9 -> 0.00 mm, vias 1 -> 0
- net /Controller/DAT1: track 71.9 -> 0.00 mm, vias 3 -> 0
- net /Controller/CS_SD: track 0.00 -> 71.8 mm, vias 0 -> 1
- net /Controller/CMD: track 65.6 -> 0.00 mm, vias 2 -> 0
- net BMS_Therm_Out: track 0.00 -> 64.1 mm, vias 0 -> 1
- net PAC2_1: track 0.00 -> 61.5 mm, vias 0 -> 1
- net /Controller/SD_MOSI: track 0.00 -> 57.1 mm, vias 0 -> 1
- net /Controller/DAT3: track 56.3 -> 0.00 mm, vias 1 -> 0
- net PAC1_2: track 0.00 -> 54.7 mm
- net PAC1_1: track 0.00 -> 52.7 mm
- net /Controller/DAT2: track 51.0 -> 0.00 mm, vias 1 -> 0
- net /Controller/SD_MISO: track 0.00 -> 49.2 mm, vias 0 -> 1
- net PAC2_2: track 0.00 -> 39.5 mm
- net /Controller/BRAKE_CTRL: track 136.1 -> 107.5 mm
- net /Controller/SD_CLK: track 68.2 -> 47.2 mm
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Other:
- board size 139 x 104.8 mm -> 138.3 x 104.8 mm
