File: Rear-Control-Board/rear-control-board-Design/Controller.kicad_sch (KiCad schematic)
At the start: 12 parts, among them J7 Micro_SD_Card, U1 Dev_Board_C, U4 MAX33054EASA+T

Commit message: oops forgot to push for awile
Other:
- note added: "?"
- note removed: "DNP"
Changed lines of the file:
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@@
     (effects (font (size 1.27 1.27)) (justify left bottom))
   )
-  (text "DNP\n" (at 252.73 140.97 0)
+  (text "?" (at 253.238 140.843 0)
     (effects (font (size 1.27 1.27) bold italic) (justify left bottom))
   )

Commit message: OOPSIE
Connections:
- net BRAKE_CTRL: now also U1.27 (GPIO16); no longer U1.9 (DAC_1/ADC2_CH8/GPIO25)
- net FAN_CTRL: now also U1.33 (GPIO21); no longer U1.10 (DAC_2/ADC2_CH9/GPIO26)
- net PAC1_1: now reaches U1.11 (ADC2_CH7/GPIO27)
- net BMS_Therm_Out: now reaches U1.36 (GPIO22)
- net CLK renamed SD_CLK
- net CMD renamed CS_SD
- net CS_SD: now also J7.2 (DAT3/CD); no longer J7.3 (CMD)
- net DAT0: no longer names the net of U1.24 (ADC2_CH2/*GPIO2)
- net DAT0: no longer J7.7 (DAT0)
- net DAT1: no longer names the net of J7.8 (DAT1)
- net DAT1: no longer U1.26 (ADC2_CH0/GPIO4)
- net DAT2: no longer names the net of J7.1 (DAT2)
- net DAT2: no longer U1.13 (*MTDI/GPIO12/ADC2_CH5)
- net DAT3 renamed SD_MOSI
- net SD_MOSI: now also J7.3 (CMD); no longer J7.2 (DAT3/CD)
- new net PAC1_2: U1.10 (DAC_2/ADC2_CH9/GPIO26)
- new net PAC2_1: U1.9 (DAC_1/ADC2_CH8/GPIO25)
- new net PAC2_2: U1.26 (ADC2_CH0/GPIO4)
- new net SD_MISO: J7.7 (DAT0), U1.13 (*MTDI/GPIO12/ADC2_CH5)
- no-connect marks 0 -> 2
Changed lines of the file:
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@@
   (junction (at 28.956 43.942) (diameter 0) (color 0 0 0 0)
   )
+  (junction (at 61.849 56.642) (diameter 0) (color 0 0 0 0)
+  )
   (junction (at 42.799 48.895) (diameter 0) (color 0 0 0 0)
   )
@@
   (junction (at 47.879 51.435) (diameter 0) (color 0 0 0 0)
   )
+  (junction (at 61.976 56.642) (diameter 0) (color 0 0 0 0)
+  )
   (junction (at 33.909 46.482) (diameter 0) (color 0 0 0 0)
   )
-  (junction (at 61.849 56.642) (diameter 0) (color 0 0 0 0)
-  )
   (junction (at 248.92 144.145) (diameter 0) (color 0 0 0 0)
   )
@@
   (junction (at 248.92 136.525) (diameter 0) (color 0 0 0 0)
   )
-  (wire (pts (xy 61.849 56.642) (xy 84.582 56.642))
+  (no_connect (at 101.346 134.747))
+  (no_connect (at 101.346 152.527))
+  (wire (pts (xy 61.976 56.642) (xy 84.582 56.642))
     (stroke (width 0) (type default) (color 0 0 0 0))
   )
@@
     (stroke (width 0) (type default) (color 0 0 0 0))
   )
+  (wire (pts (xy 61.976 55.753) (xy 61.976 56.642))
+    (stroke (width 0) (type default) (color 0 0 0 0))
+  )
   (wire (pts (xy 198.12 128.905) (xy 203.2 128.905))
     (stroke (width 0) (type default) (color 0 0 0 0))
@@
     (stroke (width 0) (type default) (color 0 0 0 0))
   )
-  (wire (pts (xy 61.849 55.753) (xy 61.849 56.642))
-    (stroke (width 0) (type default) (color 0 0 0 0))
-  )
   (wire (pts (xy 63.119 51.435) (xy 47.879 51.435))
     (stroke (width 0) (type default) (color 0 0 0 0))
@@
     (stroke (width 0) (type default) (color 0 0 0 0))
   )
+  (wire (pts (xy 84.582 54.102) (xy 56.769 54.102))
+    (stroke (width 0) (type default) (color 0 0 0 0))
+  )
+  (wire (pts (xy 265.684 79.121) (xy 264.414 79.121))
+    (stroke (width 0) (type default) (color 0 0 0 0))
+  )
+  (wire (pts (xy 56.769 54.102) (xy 56.769 58.547))
+    (stroke (width 0) (type default) (color 0 0 0 0))
+  )
+  (wire (pts (xy 227.584 76.581) (xy 227.584 78.486))
+    (stroke (width 0) (type default) (color 0 0 0 0))
+  )
   (wire (pts (xy 61.849 56.642) (xy 61.849 58.547))
     (stroke (width 0) (type default) (color 0 0 0 0))
   )
-  (wire (pts (xy 84.582 54.102) (xy 56.769 54.102))
-    (stroke (width 0) (type default) (color 0 0 0 0))
-  )
-  (wire (pts (xy 265.684 79.121) (xy 264.414 79.121))
-    (stroke (width 0) (type default) (color 0 0 0 0))
-  )
-  (wire (pts (xy 56.769 54.102) (xy 56.769 58.547))
-    (stroke (width 0) (type default) (color 0 0 0 0))
-  )
-  (wire (pts (xy 227.584 76.581) (xy 227.584 78.486))
-    (stroke (width 0) (type default) (color 0 0 0 0))
-  )
   (wire (pts (xy 71.755 49.022) (xy 59.309 48.895))
     (stroke (width 0) (type default) (color 0 0 0 0))
   )
   (wire (pts (xy 248.92 144.145) (xy 250.825 144.145))
+    (stroke (width 0) (type default) (color 0 0 0 0))
+  )
+  (wire (pts (xy 61.849 56.642) (xy 61.976 56.642))
     (stroke (width 0) (type default) (color 0 0 0 0))
   )
@@
     (effects (font (size 1.27 1.27)) (justify left bottom))
   )
-  (label "DAT2" (at 84.582 69.342 180)
+  (label "SD_MISO" (at 84.582 69.342 180)
     (effects (font (size 1.27 1.27)) (justify right bottom))
   )
@@
     (effects (font (size 1.27 1.27)) (justify right bottom))
   )
-  (label "DAT0" (at 101.346 137.287 0)
-    (effects (font (size 1.27 1.27)) (justify left bottom))
-  )
-  (label "DAT2" (at 101.346 152.527 0)
-    (effects (font (size 1.27 1.27)) (justify left bottom))
-  )
-  (label "DAT3" (at 101.346 149.987 0)
-    (effects (font (size 1.27 1.27)) (justify left bottom))
-  )
   (label "TEMP_WATER_OUT" (at 243.459 83.566 180)
     (effects (font (size 1.27 1.27)) (justify right bottom))
   )
-  (label "DAT3" (at 84.582 74.422 180)
-    (effects (font (size 1.27 1.27)) (justify right bottom))
-  )
-  (label "DAT1" (at 101.346 134.747 0)
-    (effects (font (size 1.27 1.27)) (justify left bottom))
-  )
   (label "TEMP_WATER_IN" (at 154.432 64.262 0)
     (effects (font (size 1.27 1.27)) (justify left bottom))
   )
-  (label "CMD" (at 154.432 76.962 0)
+  (label "CS_SD" (at 154.432 76.962 0)
     (effects (font (size 1.27 1.27)) (justify left bottom))
   )
@@
     (effects (font (size 1.27 1.27)) (justify left bottom))
   )
-  (label "CLK" (at 101.346 142.367 0)
-    (effects (font (size 1.27 1.27)) (justify left bottom))
-  )
-  (label "CMD" (at 101.346 147.447 0)
+  (label "SD_MOSI" (at 84.582 74.422 180)
+    (effects (font (size 1.27 1.27)) (justify right bottom))
+  )
+  (label "SD_CLK" (at 101.346 142.367 0)
     (effects (font (size 1.27 1.27)) (justify left bottom))
   )
@@
     (effects (font (size 1.27 1.27)) (justify left bottom))
   )
-  (label "DAT0" (at 154.432 74.422 0)
-    (effects (font (size 1.27 1.27)) (justify left bottom))
+  (label "SD_CLK" (at 84.582 66.802 180)
+    (effects (font (size 1.27 1.27)) (justify right bottom))
   )
   (label "TEMP_WATER_OUT" (at 154.432 71.882 0)
     (effects (font (size 1.27 1.27)) (justify left bottom))
   )
-  (label "CLK" (at 84.582 66.802 180)
-    (effects (font (size 1.27 1.27)) (justify right bottom))
-  )
-  (label "DAT1" (at 154.432 69.342 0)
+  (label "SD_MISO" (at 101.346 137.287 0)
+    (effects (font (size 1.27 1.27)) (justify left bottom))
+  )
+  (label "CS_SD" (at 101.346 149.987 0)
     (effects (font (size 1.27 1.27)) (justify left bottom))
   )
@@
     (effects (font (size 1.27 1.27)) (justify left bottom))
   )
+  (label "SD_MOSI" (at 101.346 147.447 0)
+    (effects (font (size 1.27 1.27)) (justify left bottom))
+  )
+  (global_label "PAC2_1" (shape input) (at 84.582 59.182 180) (fields_autoplaced)
+    (effects (font (size 1.27 1.27)) (justify right))
+    (property "Intersheet References" "${INTERSHEET_REFS}" (id 0) (at 75.2426 59.2614 0)
+      (effects (font (size 1.27 1.27)) (justify right) hide)
+    )
+  )
+  (global_label "PAC2_2" (shape input) (at 154.432 69.342 0) (fields_autoplaced)
+    (effects (font (size 1.27 1.27)) (justify left))
+    (property "Intersheet References" "${INTERSHEET_REFS}" (id 0) (at 163.7714 69.2626 0)
+      (effects (font (size 1.27 1.27)) (justify left) hide)
+    )
+  )
+  (global_label "PAC1_1" (shape input) (at 84.582 64.262 180) (fields_autoplaced)
+    (effects (font (size 1.27 1.27)) (justify right))
+    (property "Intersheet References" "${INTERSHEET_REFS}" (id 0) (at 75.2426 64.3414 0)
+      (effects (font (size 1.27 1.27)) (justify right) hide)
+    )
+  )
+  (global_label "PAC1_2" (shape input) (at 84.582 61.722 180) (fields_autoplaced)
+    (effects (font (size 1.27 1.27)) (justify right))
+    (property "Intersheet References" "${INTERSHEET_REFS}" (id 0) (at 75.2426 61.8014 0)
+      (effects (font (size 1.27 1.27)) (justify right) hide)
+    )
+  )
+  (global_label "BMS_Therm_Out" (shape input) (at 154.432 43.942 0) (fields_autoplaced)
+    (effects (font (size 1.27 1.27)) (justify left))
+    (property "Intersheet References" "${INTERSHEET_REFS}" (id 0) (at 171.5124 43.8626 0)
+      (effects (font (size 1.27 1.27)) (justify left) hide)
+    )
+  )
   (hierarchical_label "WHEEL_L" (shape input) (at 28.829 43.18 0)
     (effects (font (size 1.27 1.27)) (justify left))
   )
+  (hierarchical_label "BRAKE_CTRL" (shape output) (at 154.432 66.802 0)
+    (effects (font (size 1.27 1.27)) (justify left))
+  )
   (hierarchical_label "PUMP_CTRL" (shape output) (at 154.432 59.182 0)
     (effects (font (size 1.27 1.27)) (justify left))
@@
     (effects (font (size 1.27 1.27)) (justify right))
   )
-  (hierarchical_label "BRAKE_CTRL" (shape output) (at 84.582 59.182 180)
-    (effects (font (size 1.27 1.27)) (justify right))
-  )
   (hierarchical_label "CAN_N" (shape output) (at 253.365 142.875 0)
     (effects (font (size 1.27 1.27)) (justify left))
   )
+  (hierarchical_label "FAULT_BMS" (shape input) (at 61.976 55.753 0)
+    (effects (font (size 1.27 1.27)) (justify left))
+  )
   (hierarchical_label "FAULT_IMD" (shape input) (at 56.769 53.213 0)
     (effects (font (size 1.27 1.27)) (justify left))
   )
-  (hierarchical_label "FAULT_BMS" (shape input) (at 61.849 55.753 0)
-    (effects (font (size 1.27 1.27)) (justify left))
-  )
   (hierarchical_label "SUSPENSION_R" (shape input) (at 47.879 50.8 0)
     (effects (font (size 1.27 1.27)) (justify left))
   )
-  (hierarchical_label "FAN_CTRL" (shape output) (at 84.582 61.722 180)
-    (effects (font (size 1.27 1.27)) (justify right))
-  )
   (hierarchical_label "WATER_IN+" (shape input) (at 264.414 79.121 180)
     (effects (font (size 1.27 1.27)) (justify right))
   )
+  (hierarchical_label "FAN_CTRL" (shape output) (at 154.432 51.562 0)
+    (effects (font (size 1.27 1.27)) (justify left))
+  )
   (hierarchical_label "WATER_IN-" (shape input) (at 264.414 84.201 180)

Commit message: end of year DUMP
Other:
- moved on the sheet: C12, C8, D9, R4, R6, R7, U4
