File: Rear-Control-Board/rear-control-board-Design/FET_OUTPUT.kicad_sch (KiCad schematic)
At the start: 6 parts, among them Q2 PSMN5R2-60YL, Q3 PSMN5R2-60YL, Q4 PSMN5R2-60YL

Commit message: V3
Parts:
- removed Q2, Q3, Q4: PSMN5R2-60YL, Package_TO_SOT_SMD:LFPAK56, symbol Transistor_FET:PSMN5R2-60YL
- added K4, K5, K6: G5V-1, Relay_THT:Relay_SPDT_Omron_G5V-1, symbol Relay:G5V-1
Connections:
- net BRAKE_12V: now also K6.10
- net BRAKE_CTRL: now also K6.2
- net FAN_12V: now also K4.10
- net FAN_CTRL: now also K4.2
- net GND: now also K4.5, K4.6, K4.9, K5.5, K5.6, K5.9, K6.5, K6.6, K6.9
- net PUMP_12V: now also K5.10
- net PUMP_CTRL: now also K5.2
- no-connect marks 0 -> 2
