File: Rear-Control-Board/rear-control-board-Design/rear-control-board.kicad_sch (KiCad schematic)
At the start: 16 parts, among them J1 Conn_01x23, J2 Conn_01x23, J3 Conn_01x08, J6 Conn_01x02, K1 T9VV1K15-12S, U2 TS2940CP33 ROG

Commit message: oops forgot to push for awile
Other:
- note added: "12/20/2022 | 22.020 | C.Grund"
- note added: "Rear Control Board Functions: CAN, Wheel Speed, Dampers, Fan, Pump, Brake, Main Power Fuses, BRB I/O - CAN from rinehart to HVB CAN is temrinated on BMS (start of line) End of line is the Rear"
- note removed: "01/20/2022 | 22.020 | G.Spearing"
- note removed: "Rear Control Board Functions: CAN, Wheel Speed, Dampers, Fan, Pump, Brake, Main Power Fuses, BRB I/O - CAN from rinehart to HVB CAN is temrinated on Rineart (start of line) End of line is the Pacman Side 2"
Changed lines of the file:
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@@
     (effects (font (size 1.27 1.27)) (justify left bottom))
   )
-  (text "01/20/2022    |    22.020    |    G.Spearing" (at 208.28 194.31 0)
+  (text "12/20/2022    |    22.020    |    C.Grund" (at 208.28 194.31 0)
     (effects (font (size 1.27 1.27)) (justify left bottom))
   )
-  (text "Rear Control Board\nFunctions: CAN, Wheel Speed, Dampers, Fan, Pump, Brake, Main Power Fuses, BRB I/O\n- CAN from rinehart to HVB\nCAN is temrinated on Rineart (start of line)\nEnd of line is the Pacman Side 2"
+  (text "Rear Control Board\nFunctions: CAN, Wheel Speed, Dampers, Fan, Pump, Brake, Main Power Fuses, BRB I/O\n- CAN from rinehart to HVB\nCAN is temrinated on BMS (start of line)\nEnd of line is the Rear"
     (at 178.435 177.165 0)
     (effects (font (size 1.27 1.27)) (justify left bottom))

Commit message: V3
Parts:
- removed U2: TS2940CP33 ROG, Package_TO_SOT_SMD:TO-252-2, symbol Regulator_Linear:NCP1117-5.0_TO252
- added U2: TS2940CP33_ROG, Package_TO_SOT_SMD:TO-252-2, symbol AERO_Symbols:TS2940CP33_ROG
Connections:
- net GND: now also U2.2 (GND)
- net INT_12V: now also U2.1 (VI)
- net VDD: now also U2.3 (Vo)
- net BATT_12V renamed BATT_12

Commit message: OOPSIE
Connections:
- net PAC1_1: now reaches J2.11 (Pin_11)
- net PAC1_2: now reaches J2.12 (Pin_12)
- net PAC2_1: now reaches J2.13 (Pin_13)
- net PAC2_2: now reaches J2.14 (Pin_14)
- net BMS_Therm_Out: now reaches J2.3 (Pin_3)
Changed lines of the file:
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@@
+    (stroke (width 0) (type default) (color 0 0 0 0))
+  )
+  (wire (pts (xy 42.545 106.68) (xy 24.13 106.68))
     (stroke (width 0) (type default) (color 0 0 0 0))
   )
@@
     (stroke (width 0) (type default) (color 0 0 0 0))
   )
+  (wire (pts (xy 44.45 127) (xy 24.13 127))
+    (stroke (width 0) (type default) (color 0 0 0 0))
+  )
   (wire (pts (xy 44.45 124.46) (xy 44.45 121.92))
     (stroke (width 0) (type default) (color 0 0 0 0))
@@
     (stroke (width 0) (type default) (color 0 0 0 0))
   )
+  (wire (pts (xy 44.45 132.08) (xy 24.13 132.08))
+    (stroke (width 0) (type default) (color 0 0 0 0))
+  )
   (wire (pts (xy 141.224 175.768) (xy 147.574 175.768))
     (stroke (width 0) (type default) (color 0 0 0 0))
@@
     (stroke (width 0) (type default) (color 0 0 0 0))
   )
-  (wire (pts (xy 43.307 127) (xy 24.13 127))
-    (stroke (width 0) (type default) (color 0 0 0 0))
-  )
   (wire (pts (xy 89.535 59.69) (xy 89.535 62.23))
     (stroke (width 0) (type default) (color 0 0 0 0))
@@
     (stroke (width 0) (type default) (color 0 0 0 0))
   )
+  (wire (pts (xy 44.45 129.54) (xy 24.13 129.54))
+    (stroke (width 0) (type default) (color 0 0 0 0))
+  )
   (wire (pts (xy 110.109 175.768) (xy 117.221 175.768))
     (stroke (width 0) (type default) (color 0 0 0 0))
@@
   )
   (wire (pts (xy 24.13 154.94) (xy 44.45 154.94))
+    (stroke (width 0) (type default) (color 0 0 0 0))
+  )
+  (wire (pts (xy 44.45 134.62) (xy 24.13 134.62))
     (stroke (width 0) (type default) (color 0 0 0 0))
   )
@@
     )
   )
+  (global_label "PAC1_2" (shape input) (at 44.45 129.54 0) (fields_autoplaced)
+    (effects (font (size 1.27 1.27)) (justify left))
+    (property "Intersheet References" "${INTERSHEET_REFS}" (id 0) (at 53.7894 129.4606 0)
+      (effects (font (size 1.27 1.27)) (justify left) hide)
+    )
+  )
+  (global_label "PAC1_1" (shape input) (at 44.45 127 0) (fields_autoplaced)
+    (effects (font (size 1.27 1.27)) (justify left))
+    (property "Intersheet References" "${INTERSHEET_REFS}" (id 0) (at 53.7894 126.9206 0)
+      (effects (font (size 1.27 1.27)) (justify left) hide)
+    )
+  )
+  (global_label "BMS_Therm_Out" (shape input) (at 42.545 106.68 0) (fields_autoplaced)
+    (effects (font (size 1.27 1.27)) (justify left))
+    (property "Intersheet References" "${INTERSHEET_REFS}" (id 0) (at 59.6254 106.6006 0)
+      (effects (font (size 1.27 1.27)) (justify left) hide)
+    )
+  )
+  (global_label "PAC2_2" (shape input) (at 44.45 134.62 0) (fields_autoplaced)
+    (effects (font (size 1.27 1.27)) (justify left))
+    (property "Intersheet References" "${INTERSHEET_REFS}" (id 0) (at 53.7894 134.5406 0)
+      (effects (font (size 1.27 1.27)) (justify left) hide)
+    )
+  )
+  (global_label "PAC2_1" (shape input) (at 44.45 132.08 0) (fields_autoplaced)
+    (effects (font (size 1.27 1.27)) (justify left))
+    (property "Intersheet References" "${INTERSHEET_REFS}" (id 0) (at 53.7894 132.0006 0)
+      (effects (font (size 1.27 1.27)) (justify left) hide)
+    )
+  )

Commit message: end of year DUMP
Other:
- moved on the sheet: C1, C4, D1, D10, D11, D12, D8, H1, H2, J1, J2, J3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
