File: Therm Board/Themal expansion/Themal expansion.kicad_sch (KiCad schematic)
At the start: 8 parts

Commit message: OOPSIE
Parts:
- removed IC? (x5): CD74HC4051QPWRQ1, SOP65P640X120-16N, symbol CD74HC4051QPWRQ1:CD74HC4051QPWRQ1
- removed J? (x2): Conn_01x23, symbol Connector_Generic:Conn_01x23
- added J?: Conn_01x08, symbol Connector_Generic:Conn_01x08
Connections:
- new net +12V: J?.8 (Pin_8)
- new net BMS_OUT: J?.2 (Pin_2)
- new net GND: J?.1 (Pin_1)
- new net PAC1_1: J?.7 (Pin_7)
- new net PAC1_2: J?.6 (Pin_6)
- new net PAC2_1: J?.5 (Pin_5)
- new net PAC2_2: J?.4 (Pin_4)
