File: Documentation/Charger/Charger.kicad_sch (KiCad schematic)
At the start: 14 parts

Commit message: documentation
Parts:
- J?: value Orion2 BMS -> n-BMS
Connections:
- net at U?.: now also F?.2; no longer U?.
- net Cell_Voltages renamed IP
- net Temp_Sensors renamed IM
- new net: F?.1, U?., U?. (IP)
- new net: BT?.2 (-), U?., U?. (IP)
- new net: U?., U?.
- new net: U?., U?. (GND)
Changed lines of the file:
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@@
     (effects (font (size 1.27 1.27)) (justify left bottom))
   )
-  (label "Cell_Voltages" (at 50.165 82.55 0)
+  (label "IP" (at 50.165 82.55 0)
     (effects (font (size 1.27 1.27)) (justify left bottom))
   )
@@
     (effects (font (size 1.27 1.27)) (justify left bottom))
   )
-  (label "Temp_Sensors" (at 50.165 80.01 0)
+  (label "IM" (at 50.165 80.01 0)
     (effects (font (size 1.27 1.27)) (justify left bottom))
   )
@@
       (effects (font (size 1.27 1.27)) hide)
     )
-    (property "Value" "Orion2 BMS" (id 1) (at 36.83 90.17 0))
+    (property "Value" "n-BMS" (id 1) (at 36.83 90.17 0))
     (property "Footprint" "" (id 2) (at 44.45 90.17 0)
       (effects (font (size 1.27 1.27)) hide)
@@
     )
     (path "/7599133e-c681-4202-85d9-c20dac196c64"
-      (reference "J?") (unit 1) (value "Orion2 BMS") (footprint "")
+      (reference "J?") (unit 1) (value "n-BMS") (footprint "")
     )
     (path "/cf18cdc4-21f0-43b7-ba25-4e573c33e3c5"

Commit message: end of year DUMP
Parts:
- removed F?: 20A, symbol Device:Fuse
- added J?: Conn_01x03, symbol Connector_Generic:Conn_01x03
- added J?: Conn_01x08, symbol Connector_Generic:Conn_01x08
- K?: value T9VV1K15-12S -> (none)
Connections:
- net Charge_Power: now also BT?.1 (+), J?.2 (Pin_2)
- net GND: now also J?.1 (Pin_1)
- net at U?.: now also U?.; no longer U?.
- removed net Always_On_Power: BT?.1 (+), J?.1 (Pin_1), J?.2 (Pin_2)
- net IM renamed SSOK
- net SSOK: no longer U?. (IP)
- net IP: no longer names the net of J?.1 (Pin_1)
- net IP: no longer U?. (IP)
- new net: F?.1, U?., U?. (Bat-)
- new net: BT?.2 (-), U?., U?. (Bat-)
- new net: U?., U?.
- new net: U?., U?. (GND) (x2)
- new net +12V: J?.8 (Pin_8)
- new net Main AIR: J?.7 (Pin_7), U?. (Bat-)
- new net Precharge: J?.1 (Pin_1), J?.5 (Pin_5)
- new net Secondary AIR: J?.6 (Pin_6), U?. (Bat-)
- new net Temp1: J?.2 (Pin_2), J?.4 (Pin_4)
- new net Temp2: J?.3 (Pin_3), J?.3 (Pin_3)
