File: Documentation/Shut off circuitry/Shut off circuitry.kicad_sch (KiCad schematic)
At the start: 26 parts

Commit message: end of year DUMP
Parts:
- removed SW? (x2): Pack Interlock, symbol Switch:SW_SPST
Connections:
- net at K?.6, K?.6, SW?.2 (B): now also J?.1 (Pin_1)
- net at K?.1, K?.14: now also SW?.1 (A)
Other:
- note added: "AMS: Accumulator Managment system (Orion 2) HIGH FAULT LOW CLEAR IMD: Isolation Monitoring Device (Bender IR155-3024) LOW FAULT HIGH CLEAR Temperature Monitoring controlled by AMS Fault"
- note removed: "AMS: Accumulator Managment system (Orion 2) IMD: Isolation Monitoring Device (Bender IR155-3024) Temperature Monitoring controlled by AMS Fault"
Changed lines of the file:
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@@
 (kicad_sch (version 20211123) (generator eeschema)
-  (paper "A4")
-  (junction (at 198.12 59.69) (diameter 0) (color 0 0 0 0)
-  )
+  (paper "A")
   (junction (at 38.1 118.11) (diameter 0) (color 0 0 0 0)
   )
@@
   (junction (at 209.55 142.24) (diameter 0) (color 0 0 0 0)
   )
+  (junction (at 198.12 90.9828) (diameter 0) (color 0 0 0 0)
+  )
   (junction (at 213.36 95.25) (diameter 0) (color 0 0 0 0)
   )
@@
     (stroke (width 0) (type default) (color 0 0 0 0))
   )
-  (wire (pts (xy 198.12 49.53) (xy 198.12 59.69))
-    (stroke (width 0) (type default) (color 0 0 0 0))
-  )
   (wire (pts (xy 171.45 27.94) (xy 198.12 27.94))
     (stroke (width 0) (type default) (color 0 0 0 0))
@@
     (stroke (width 0) (type default) (color 0 0 0 0))
   )
-  (wire (pts (xy 198.12 59.69) (xy 199.39 59.69))
-    (stroke (width 0) (type default) (color 0 0 0 0))
-  )
   (wire (pts (xy 195.58 116.84) (xy 195.58 97.79))
     (stroke (width 0) (type default) (color 0 0 0 0))
@@
     (stroke (width 0) (type default) (color 0 0 0 0))
   )
+  (wire (pts (xy 198.12 90.9828) (xy 198.12 97.79))
+    (stroke (width 0) (type default) (color 0 0 0 0))
+  )
   (wire (pts (xy 229.87 115.57) (xy 229.87 95.25))
     (stroke (width 0) (type default) (color 0 0 0 0))
@@
     (stroke (width 0) (type default) (color 0 0 0 0))
   )
-  (wire (pts (xy 198.12 27.94) (xy 198.12 29.21))
+  (wire (pts (xy 198.12 27.94) (xy 198.12 64.77))
     (stroke (width 0) (type default) (color 0 0 0 0))
   )
@@
     (stroke (width 0) (type default) (color 0 0 0 0))
   )
+  (wire (pts (xy 190.8048 90.9828) (xy 198.12 90.9828))
+    (stroke (width 0) (type default) (color 0 0 0 0))
+  )
   (wire (pts (xy 66.04 118.11) (xy 38.1 118.11))
     (stroke (width 0) (type default) (color 0 0 0 0))
@@
     (stroke (width 0) (type default) (color 0 0 0 0))
   )
-  (wire (pts (xy 198.12 59.69) (xy 198.12 64.77))
+  (wire (pts (xy 198.12 90.17) (xy 198.12 90.9828))
     (stroke (width 0) (type default) (color 0 0 0 0))
   )
@@
   )
   (wire (pts (xy 203.2 119.38) (xy 193.04 119.38))
-    (stroke (width 0) (type default) (color 0 0 0 0))
-  )
-  (wire (pts (xy 198.12 90.17) (xy 198.12 97.79))
     (stroke (width 0) (type default) (color 0 0 0 0))
   )
@@
     (effects (font (size 1.27 1.27)) (justify left bottom))
   )
-  (text "AMS: Accumulator Managment system (Orion 2)\nIMD: Isolation Monitoring Device (Bender IR155-3024)\n\nTemperature Monitoring controlled by AMS Fault\n"
+  (text "AMS: Accumulator Managment system (Orion 2) HIGH FAULT LOW CLEAR\nIMD: Isolation Monitoring Device (Bender IR155-3024) LOW FAULT HIGH CLEAR\n\nTemperature Monitoring controlled by AMS Fault\n"
     (at 88.9 80.01 0)
     (effects (font (size 1.27 1.27)) (justify left bottom))
@@
     (pin "1")
   )
-  (symbol (lib_id "Switch:SW_SPST") (at 198.12 34.29 270) (unit 1)
-    (in_bom yes) (on_board yes) (fields_autoplaced)
-    (property "Reference" "SW?" (id 0) (at 200.533 33.3815 90)
-      (effects (font (size 1.27 1.27)) (justify left) hide)
-    )
-    (property "Value" "Pack Interlock" (id 1) (at 200.533 34.769 90)
-      (effects (font (size 1.27 1.27)) (justify left))
-    )
-    (property "Footprint" "" (id 2) (at 198.12 34.29 0)
-      (effects (font (size 1.27 1.27)) hide)
-    )
-    (property "Datasheet" "~" (id 3) (at 198.12 34.29 0)
-      (effects (font (size 1.27 1.27)) hide)
-    )
-    (pin "1")
-    (pin "2")
-  )
   (symbol (lib_id "Connector_Generic:Conn_01x01") (at 229.87 92.71 0) (unit 1)
     (in_bom yes) (on_board yes) (fields_autoplaced)
@@
     )
     (pin "1")
-  )
-  (symbol (lib_id "Switch:SW_SPST") (at 198.12 44.45 270) (unit 1)
-    (in_bom yes) (on_board yes) (fields_autoplaced)
-    (property "Reference" "SW?" (id 0) (at 200.533 43.5415 90)
-      (effects (font (size 1.27 1.27)) (justify left) hide)
-    )
-    (property "Value" "Pack Interlock" (id 1) (at 200.533 44.929 90)
-      (effects (font (size 1.27 1.27)) (justify left))
-    )
-    (property "Footprint" "" (id 2) (at 198.12 44.45 0)
-      (effects (font (size 1.27 1.27)) hide)
-    )
-    (property "Datasheet" "~" (id 3) (at 198.12 44.45 0)
-      (effects (font (size 1.27 1.27)) hide)
-    )
-    (pin "1")
-    (pin "2")
   )
   (symbol (lib_id "Switch:SW_SPST") (at 38.1 45.72 90) (unit 1)
@@
     (pin "2")
   )
-  (symbol (lib_id "Connector_Generic:Conn_01x01") (at 204.47 59.69 0) (unit 1)
-    (in_bom yes) (on_board yes) (fields_autoplaced)
-    (property "Reference" "J?" (id 0) (at 203.5615 57.658 90)
-      (effects (font (size 1.27 1.27)) (justify left) hide)
-    )
-    (property "Value" "ESOK" (id 1) (at 206.502 60.169 0)
-      (effects (font (size 1.27 1.27)) (justify left))
-    )
-    (property "Footprint" "" (id 2) (at 204.47 59.69 0)
-      (effects (font (size 1.27 1.27)) hide)
-    )
-    (property "Datasheet" "~" (id 3) (at 204.47 59.69 0)
+  (symbol (lib_id "Connector_Generic:Conn_01x01") (at 185.7248 90.9828 180) (unit 1)
+    (in_bom yes) (on_board yes) (fields_autoplaced)
+    (property "Reference" "J?" (id 0) (at 186.6333 93.0148 90)
+      (effects (font (size 1.27 1.27)) (justify left) hide)
+    )
+    (property "Value" "ESOK" (id 1) (at 185.7248 86.7156 0))
+    (property "Footprint" "" (id 2) (at 185.7248 90.9828 0)
+      (effects (font (size 1.27 1.27)) hide)
+    )
+    (property "Datasheet" "~" (id 3) (at 185.7248 90.9828 0)
       (effects (font (size 1.27 1.27)) hide)
     )
@@
       (reference "R?") (unit 1) (value "R") (footprint "")
     )
-    (path "/3156380f-46fe-42b0-adf2-d39b5b26f29a"
-      (reference "SW?") (unit 1) (value "Pack Interlock") (footprint "")
-    )
     (path "/4b98a9d7-d892-4691-be54-bdfe93e8941c"
       (reference "SW?") (unit 1) (value "Cockpit BRB") (footprint "")
@@
       (reference "SW?") (unit 1) (value "GLVMS") (footprint "")
     )
-    (path "/73f890cd-9899-4131-b70d-d26b840fea95"
-      (reference "SW?") (unit 1) (value "Pack Interlock") (footprint "")
-    )
     (path "/779a10b6-96e5-4987-b384-b8f010de3ecb"
