File: HVB High Voltage Board V1/high-voltage-board.kicad_sch (KiCad schematic)
At the start: 17 parts, among them J1 Conn_01x23, J11 HV-, J2 Conn_01x02, J3 HV+, J4 HV-, J5 HV+, J6 HV-, J8 HV+, J9 Bender-LV

Commit message: end of year DUMP
Other:
- moved on the sheet: F1, H1, H2, H3, H4
Changed lines of the file:
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@@
 (kicad_sch (version 20211123) (generator eeschema)
-  (paper "A4")
+  (paper "A")
   (junction (at 35.56 177.165) (diameter 0) (color 0 0 0 0)
   )
@@
     (stroke (width 0) (type default) (color 0 0 0 0))
   )
-  (wire (pts (xy 113.665 186.69) (xy 119.38 186.69))
+  (wire (pts (xy 136.9822 147.2692) (xy 142.6972 147.2692))
     (stroke (width 0) (type default) (color 0 0 0 0))
   )
@@
     (stroke (width 0) (type default) (color 0 0 0 0))
   )
-  (wire (pts (xy 170.815 187.96) (xy 158.115 187.96))
+  (wire (pts (xy 194.1322 148.5392) (xy 181.4322 148.5392))
     (stroke (width 0) (type default) (color 0 0 0 0))
   )
@@
     (stroke (width 0) (type default) (color 0 0 0 0))
   )
-  (wire (pts (xy 126.365 189.23) (xy 133.35 189.23))
+  (wire (pts (xy 149.6822 149.8092) (xy 156.6672 149.8092))
     (stroke (width 0) (type default) (color 0 0 0 0))
   )
@@
     (stroke (width 0) (type default) (color 0 0 0 0))
   )
-  (wire (pts (xy 127 186.69) (xy 133.35 186.69))
+  (wire (pts (xy 150.3172 147.2692) (xy 156.6672 147.2692))
     (stroke (width 0) (type default) (color 0 0 0 0))
   )
@@
     (effects (font (size 1.27 1.27)) (justify left bottom))
   )
-  (text "Global nets connected to this sheet: \n12V, GND" (at 133.35 177.165 0)
+  (text "Global nets connected to this sheet: \n12V, GND" (at 160.2994 181.0004 0)
     (effects (font (size 1.27 1.27)) (justify left bottom))
   )
@@
   )
   (text "Board Function: \n- CAN IN/OUT from RCB to DCB and Pack 1\n- Vicor DC/DC \n- TSMP\n- BMS Current\n- STM32 (Precharge)\n- TSAL\n- IMD"
-    (at 177.8 182.245 0)
+    (at 216.154 187.8584 0)
     (effects (font (size 1.27 1.27)) (justify left bottom))
   )
@@
     (effects (font (size 1.27 1.27)) (justify left bottom))
   )
-  (text "12v comes from DC/DC not GLV" (at 132.715 170.815 0)
+  (text "12v comes from DC/DC not GLV" (at 159.6644 174.6504 0)
     (effects (font (size 1.27 1.27) bold italic) (justify left bottom))
   )
@@
     (effects (font (size 1.27 1.27) (thickness 0.254) bold italic) (justify left bottom))
   )
-  (label "HV-" (at 126.365 189.23 0)
+  (label "HV-" (at 149.6822 149.8092 0)
     (effects (font (size 1.27 1.27)) (justify left bottom))
   )
@@
     (effects (font (size 1.27 1.27)) (justify left bottom))
   )
-  (label "TSAL_GND" (at 170.815 187.96 180)
+  (label "TSAL_GND" (at 194.1322 148.5392 180)
     (effects (font (size 1.27 1.27)) (justify right bottom))
   )
@@
     (effects (font (size 1.27 1.27)) (justify right bottom))
   )
-  (label "HV+" (at 113.665 186.69 0)
+  (label "HV+" (at 136.9822 147.2692 0)
     (effects (font (size 1.27 1.27)) (justify left bottom))
   )
@@
     (pin "1")
   )
-  (symbol (lib_id "Device:Fuse") (at 123.19 186.69 270) (unit 1)
-    (in_bom yes) (on_board yes)
-    (property "Reference" "F1" (id 0) (at 123.19 181.6862 90))
-    (property "Value" "2A" (id 1) (at 123.19 183.9976 90))
-    (property "Footprint" "Fuse:Fuseholder_Cylinder-5x20mm_Schurter_0031_8201_Horizontal_Open" (id 2) (at 123.19 184.912 90)
-      (effects (font (size 1.27 1.27)) hide)
-    )
-    (property "Datasheet" "~" (id 3) (at 123.19 186.69 0)
+  (symbol (lib_id "Device:Fuse") (at 146.5072 147.2692 270) (unit 1)
+    (in_bom yes) (on_board yes)
+    (property "Reference" "F1" (id 0) (at 146.5072 142.2654 90))
+    (property "Value" "2A" (id 1) (at 146.5072 144.5768 90))
+    (property "Footprint" "Fuse:Fuseholder_Cylinder-5x20mm_Schurter_0031_8201_Horizontal_Open" (id 2) (at 146.5072 145.4912 90)
+      (effects (font (size 1.27 1.27)) hide)
+    )
+    (property "Datasheet" "~" (id 3) (at 146.5072 147.2692 0)
       (effects (font (size 1.27 1.27)) hide)
     )
@@
     (pin "1")
   )
-  (symbol (lib_id "Mechanical:MountingHole") (at 262.255 162.56 0) (unit 1)
+  (symbol (lib_id "Mechanical:MountingHole") (at 246.7864 154.432 0) (unit 1)
     (in_bom yes) (on_board yes) (fields_autoplaced)
-    (property "Reference" "H4" (id 0) (at 264.795 161.6515 0)
-      (effects (font (size 1.27 1.27)) (justify left))
-    )
-    (property "Value" "MountingHole" (id 1) (at 264.795 164.4266 0)
-      (effects (font (size 1.27 1.27)) (justify left))
-    )
-    (property "Footprint" "MountingHole:MountingHole_3.2mm_M3" (id 2) (at 262.255 162.56 0)
-      (effects (font (size 1.27 1.27)) hide)
-    )
-    (property "Datasheet" "~" (id 3) (at 262.255 162.56 0)
-      (effects (font (size 1.27 1.27)) hide)
-    )
-  )
-  (symbol (lib_id "Mechanical:MountingHole") (at 241.935 155.575 0) (unit 1)
+    (property "Reference" "H4" (id 0) (at 249.3264 153.5235 0)
+      (effects (font (size 1.27 1.27)) (justify left))
+    )
+    (property "Value" "MountingHole" (id 1) (at 249.3264 156.2986 0)
+      (effects (font (size 1.27 1.27)) (justify left))
+    )
+    (property "Footprint" "MountingHole:MountingHole_3.2mm_M3" (id 2) (at 246.7864 154.432 0)
+      (effects (font (size 1.27 1.27)) hide)
+    )
+    (property "Datasheet" "~" (id 3) (at 246.7864 154.432 0)
+      (effects (font (size 1.27 1.27)) hide)
+    )
+  )
+  (symbol (lib_id "Mechanical:MountingHole") (at 226.4664 147.447 0) (unit 1)
     (in_bom yes) (on_board yes) (fields_autoplaced)
-    (property "Reference" "H2" (id 0) (at 244.475 154.6665 0)
-      (effects (font (size 1.27 1.27)) (justify left))
-    )
-    (property "Value" "MountingHole" (id 1) (at 244.475 157.4416 0)
-      (effects (font (size 1.27 1.27)) (justify left))
-    )
-    (property "Footprint" "MountingHole:MountingHole_3.2mm_M3" (id 2) (at 241.935 155.575 0)
-      (effects (font (size 1.27 1.27)) hide)
-    )
-    (property "Datasheet" "~" (id 3) (at 241.935 155.575 0)
+    (property "Reference" "H2" (id 0) (at 229.0064 146.5385 0)
+      (effects (font (size 1.27 1.27)) (justify left))
+    )
+    (property "Value" "MountingHole" (id 1) (at 229.0064 149.3136 0)
+      (effects (font (size 1.27 1.27)) (justify left))
+    )
+    (property "Footprint" "MountingHole:MountingHole_3.2mm_M3" (id 2) (at 226.4664 147.447 0)
+      (effects (font (size 1.27 1.27)) hide)
+    )
+    (property "Datasheet" "~" (id 3) (at 226.4664 147.447 0)
       (effects (font (size 1.27 1.27)) hide)
     )
@@
     (pin "2")
   )
-  (symbol (lib_id "Mechanical:MountingHole") (at 262.255 156.21 0) (unit 1)
+  (symbol (lib_id "Mechanical:MountingHole") (at 246.7864 148.082 0) (unit 1)
     (in_bom yes) (on_board yes) (fields_autoplaced)
-    (property "Reference" "H3" (id 0) (at 264.795 155.3015 0)
-      (effects (font (size 1.27 1.27)) (justify left))
-    )
-    (property "Value" "MountingHole" (id 1) (at 264.795 158.0766 0)
-      (effects (font (size 1.27 1.27)) (justify left))
-    )
-    (property "Footprint" "MountingHole:MountingHole_3.2mm_M3" (id 2) (at 262.255 156.21 0)
-      (effects (font (size 1.27 1.27)) hide)
-    )
-    (property "Datasheet" "~" (id 3) (at 262.255 156.21 0)
+    (property "Reference" "H3" (id 0) (at 249.3264 147.1735 0)
+      (effects (font (size 1.27 1.27)) (justify left))
+    )
+    (property "Value" "MountingHole" (id 1) (at 249.3264 149.9486 0)
+      (effects (font (size 1.27 1.27)) (justify left))
+    )
+    (property "Footprint" "MountingHole:MountingHole_3.2mm_M3" (id 2) (at 246.7864 148.082 0)
+      (effects (font (size 1.27 1.27)) hide)
+    )
+    (property "Datasheet" "~" (id 3) (at 246.7864 148.082 0)
       (effects (font (size 1.27 1.27)) hide)
     )
@@
     (pin "1")
   )
-  (symbol (lib_id "Mechanical:MountingHole") (at 241.935 162.56 0) (unit 1)
+  (symbol (lib_id "Mechanical:MountingHole") (at 226.4664 154.432 0) (unit 1)
     (in_bom yes) (on_board yes) (fields_autoplaced)
-    (property "Reference" "H1" (id 0) (at 244.475 161.6515 0)
-      (effects (font (size 1.27 1.27)) (justify left))
-    )
-    (property "Value" "MountingHole" (id 1) (at 244.475 164.4266 0)
-      (effects (font (size 1.27 1.27)) (justify left))
-    )
-    (property "Footprint" "MountingHole:MountingHole_3.2mm_M3" (id 2) (at 241.935 162.56 0)
-      (effects (font (size 1.27 1.27)) hide)
-    )
-    (property "Datasheet" "~" (id 3) (at 241.935 162.56 0)
+    (property "Reference" "H1" (id 0) (at 229.0064 153.5235 0)
+      (effects (font (size 1.27 1.27)) (justify left))
+    )
+    (property "Value" "MountingHole" (id 1) (at 229.0064 156.2986 0)
+      (effects (font (size 1.27 1.27)) (justify left))
+    )
+    (property "Footprint" "MountingHole:MountingHole_3.2mm_M3" (id 2) (at 226.4664 154.432 0)
+      (effects (font (size 1.27 1.27)) hide)
+    )
+    (property "Datasheet" "~" (id 3) (at 226.4664 154.432 0)
       (effects (font (size 1.27 1.27)) hide)
     )
@@
     )
   )
-  (sheet (at 133.35 184.15) (size 24.765 8.255) (fields_autoplaced)
+  (sheet (at 156.6672 144.7292) (size 24.765 8.255) (fields_autoplaced)
     (stroke (width 0) (type solid) (color 0 0 0 0))
     (fill (color 0 0 0 0.0000))
-    (property "Sheet name" "TSAL" (id 0) (at 133.35 183.4384 0)
+    (property "Sheet name" "TSAL" (id 0) (at 156.6672 144.0176 0)
       (effects (font (size 1.27 1.27)) (justify left bottom))
     )
-    (property "Sheet file" "TSAL.kicad_sch" (id 1) (at 133.35 192.9896 0)
+    (property "Sheet file" "TSAL.kicad_sch" (id 1) (at 156.6672 153.5688 0)
       (effects (font (size 1.27 1.27)) (justify left top))
     )
-    (pin "TSAL_GND" output (at 158.115 187.96 0)
-      (effects (font (size 1.27 1.27)) (justify right))
-    )
-    (pin "HV+" input (at 133.35 186.69 180)
-      (effects (font (size 1.27 1.27)) (justify left))
-    )
-    (pin "HV-" input (at 133.35 189.23 180)
-      (effects (font (size 1.27 1.27)) (justify left))
-    )
+    (pin "TSAL_GND" output (at 181.4322 148.5392 0)
+      (effects (font (size 1.27 1.27)) (justify right))
+    )
+    (pin "HV+" input (at 156.6672 147.2692 180)
+      (effects (font (size 1.27 1.27)) (justify left))
+    )
+    (pin "HV-" input (at 156.6672 149.8092 180)
+      (effects (font (size 1.27 1.27)) (justify left))
+    )
