File: HVB High Voltage Board V1/vicor.kicad_sch (KiCad schematic)
At the start: 15 parts, among them U7 Vicor_AERO, U8 LTV-817S, U9 TLP184

Commit message: end of year DUMP
Changed lines of the file:
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@@
 (kicad_sch (version 20211123) (generator eeschema)
-  (paper "A4")
+  (paper "A")
   (junction (at 104.14 144.78) (diameter 0) (color 0 0 0 0)
   )
@@
     (effects (font (size 1.27 1.27)) (justify left bottom))
   )
-  (text "Willem Hillier\nUVM AERO\n3/5/2019" (at 220.98 179.07 0)
+  (text "Willem Hillier\nUVM AERO\n3/5/2019" (at 161.8996 185.6232 0)
     (effects (font (size 2.54 2.54)) (justify left bottom))
   )
