File: pacman_side_2/pacman_side_2.kicad_sch (KiCad schematic)
At the start: 19 parts, among them J1 Conn_01x08, J3 Conn_01x01, J4 Conn_01x01, J5 Conn_01x01, J6 Conn_01x02, J9 JST PH, K1 G2RL, K2 G5V-1, K3 G5V-1, Q2 MMBT2222A

Commit message: end of year DUMP
Other:
- moved on the sheet: F3, J6, K3
